Commit message: Flip left LEAP mount and adjust initial pose

File: assets/robots/crx5ia_leap_paxini_left/urdf/crx5ia_leap_paxini_left.urdf (robot description, URDF)
Before this commit: robot crx5ia_leap_paxini_left, 46 links, 45 joints
Joints:
- joint flange_to_leap: origin xyz=0.037336626243399 0.047897767636037 0.140188227821871 rpy=0 -1.56 0 -> xyz=0.037336626243399 -0.047897767636037 -0.140188227821871 rpy=-3.141592653589793 1.56 0

Commit message: Restore left LEAP flange mount orientation

File: assets/robots/crx5ia_leap_paxini_left/urdf/crx5ia_leap_paxini_left.urdf (robot description, URDF)
Before this commit: robot crx5ia_leap_paxini_left, 46 links, 45 joints
Joints:
- joint flange_to_leap: origin xyz=0.037336626243399 -0.047897767636037 -0.140188227821871 rpy=-3.141592653589793 1.56 0 -> xyz=0.037336626243399 0.047897767636037 0.140188227821871 rpy=0 -1.56 0
