Commit message: Checkpoint LEAP flange remount with zero J6 initial pose
Preserve the requested two-file prototype scope. Generator, manifest and old mount test expectations remain pending synchronization; three model tests currently fail.

File: assets/robots/crx5ia_leap_paxini/urdf/crx5ia_leap_paxini.urdf (robot description, URDF)
Before this commit: robot crx5ia_leap_paxini, 46 links, 45 joints
Joints:
- joint flange_to_leap: origin xyz=0.01 0.03 0.065 rpy=0 -1.56 0 -> xyz=0.01 -0.03 -0.065 rpy=-3.141592653589793 1.56 0

Commit message: Mirror right LEAP mount XY translation

File: assets/robots/crx5ia_leap_paxini/urdf/crx5ia_leap_paxini.urdf (robot description, URDF)
Before this commit: robot crx5ia_leap_paxini, 46 links, 45 joints
Joints:
- joint flange_to_leap: origin xyz=0.01 -0.03 -0.065 rpy=-3.141592653589793 1.56 0 -> xyz=0.037336626243399 -0.047897767636037 -0.065 rpy=-3.141592653589793 1.56 0

Commit message: Revert right LEAP mount XY mirror

File: assets/robots/crx5ia_leap_paxini/urdf/crx5ia_leap_paxini.urdf (robot description, URDF)
Before this commit: robot crx5ia_leap_paxini, 46 links, 45 joints
Joints:
- joint flange_to_leap: origin xyz=0.037336626243399 -0.047897767636037 -0.065 rpy=-3.141592653589793 1.56 0 -> xyz=0.01 -0.03 -0.065 rpy=-3.141592653589793 1.56 0
