Commit message: Fix Sharpa wrist frame alignment with Quest tracking
Remove the extra 90-degree optimization-frame rotation while preserving physical mounts. Regenerate all four models and align synthetic input with the decoded Quest basis.

Add WebXR decoder-to-FK regression coverage for both hands, hand-only and arm configurations, initial wrist rotations, and finger flexion. Validation: 18 focused tests passed; user confirmed live tracking is corrected.

File: assets/robots/crx5ia_sharpa_wave_left/urdf/crx5ia_sharpa_wave_left.urdf (robot description, URDF)
Before this commit: robot crx5ia_sharpa_wave_left, 48 links, 47 joints
Joints:
- joint left_retarget_wrist_fixed: origin xyz=0 0 0 rpy=0 -1.5707963267948966 0 -> xyz=0 0 0 rpy=0 0 0

File: assets/robots/crx5ia_sharpa_wave_right/urdf/crx5ia_sharpa_wave_right.urdf (robot description, URDF)
Before this commit: robot crx5ia_sharpa_wave_right, 48 links, 47 joints
Joints:
- joint right_retarget_wrist_fixed: origin xyz=0 0 0 rpy=0 -1.5707963267948966 0 -> xyz=0 0 0 rpy=0 0 0

File: assets/robots/sharpa_wave_left/urdf/sharpa_wave_left.urdf (robot description, URDF)
Before this commit: robot sharpa_wave_left, 37 links, 36 joints
Joints:
- joint left_retarget_wrist_fixed: origin xyz=0 0 0 rpy=0 -1.5707963267948966 0 -> xyz=0 0 0 rpy=0 0 0

File: assets/robots/sharpa_wave_right/urdf/sharpa_wave_right.urdf (robot description, URDF)
Before this commit: robot sharpa_wave_right, 37 links, 36 joints
Joints:
- joint right_retarget_wrist_fixed: origin xyz=0 0 0 rpy=0 -1.5707963267948966 0 -> xyz=0 0 0 rpy=0 0 0
